Commit message: Add files via upload

File: FAR_bot-main/description/gazebo_control.xacro (robot description, xacro)
@@ -28,5 +28,5 @@
             <publish_wheel_tf>true</publish_wheel_tf>
             <odometry_frame>odom</odometry_frame>
-            <robot_base_frame>base_link</robot_base_frame>
+            <robot_base_frame>base_footprint</robot_base_frame>
         </plugin>
     </gazebo>

File: FAR_bot-main/description/robot.urdf.xacro (robot description, xacro)
@@ -10,5 +10,4 @@
         <xacro:include filename="gazebo_control.xacro" />
     </xacro:unless>
-    <!-- <xacro:include filename="gazebo_control.xacro" /> -->
     <xacro:include filename="lidar.xacro" />
 </robot>

File: FAR_bot-main/description/robot_core.xacro (robot description, xacro)
@@ -20,12 +20,12 @@
     <link name="base_link">
     </link>
-    <!-- BASE_FOOTPRINT LINK -->
+     <!-- BASE_FOOTPRINT LINK -->
+    <link name="base_footprint">
+    </link>
     <joint name="base_footprint_joint" type="fixed">
         <parent link="base_link"/>
         <child link="base_footprint"/>
-        <origin xyz="0 0 0" rpy="0 0 0"/>
+        <origin xyz="0 0 0" rpy="0 0 3.14159265359"/>
     </joint>
-    <link name="base_footprint">
-    </link>
     <!-- Chassis Link -->
     <joint name="chassis_joint" type="fixed">
@@ -73,5 +73,5 @@
         <collision>
             <geometry>
-                <cylinder radius="0.0225" length="0.018" />
+                <sphere radius="0.0225" />
             </geometry>
         </collision>
@@ -101,5 +101,5 @@
         <collision>
             <geometry>
-                <cylinder radius="0.0225" length="0.018" />
+                <sphere radius="0.0225" />
             </geometry>
         </collision>
@@ -129,5 +129,5 @@
         <collision>
             <geometry>
-                <cylinder radius="0.0225" length="0.018" />
+                <sphere radius="0.0225" />
             </geometry>
         </collision>
@@ -157,5 +157,5 @@
         <collision>
             <geometry>
-                <cylinder radius="0.0225" length="0.018" />
+                <sphere radius="0.0225" />
             </geometry>
         </collision>

File: FAR_bot-main/description/ros2_control.xacro (robot description, xacro)
@@ -5,13 +5,13 @@
             <hardware>
                 <plugin>diffdrive_arduino/DiffDriveArduino</plugin>
-                <param name="left_wheel_name">left_front_wheel_joint,left_rear_wheel_joint</param>
-                <param name="right_wheel_name">right_front_wheel_joint,right_rear_wheel_joint</param>
+                <param name="left_wheel_name">left_wheel_joint</param>
+                <param name="right_wheel_name">right_wheel_joint</param>
                 <param name="loop_rate">30</param>
                 <param name="device">/dev/ttyACM0</param>
                 <param name="baud_rate">57600</param>
                 <param name="timeout">1000</param>
-                <!-- <param name="enc_counts_per_rev">3436</param> -->
+                <param name="enc_counts_per_rev">500</param>
             </hardware>
-            <joint name="left_front_wheel_joint">
+            <joint name="left_wheel_joint">
                 <command_interface name="velocity">
                     <param name="min">-10</param>
@@ -29,5 +29,5 @@
                 <state_interface name="position"/>
             </joint>
-            <joint name="right_front_wheel_joint">
+            <joint name="right_wheel_joint">
                 <command_interface name="velocity">
                     <param name="min">-10</param>
